File: BEAPER-Nano.kicad_pcb (KiCad board)
At the start: 2 copper layers, 114.3 x 95.2 mm, 95 parts, among them CON1 Phoenix 1729160, J1 Digital, J2 Analog, J3 Conn_01x08, J4 QWIIC/JST SH, Q1 LTR-4206E, Q2 LTR-4206E, Q3 LTR-4206E, Q4 TEPT4400, SW1 RESET, SW2 SW_Push, SW3 SW_Push, SW4 SW_Push, SW5 SW_Push, U1 LM2940T-5.0, U2 74HCT541, U3 SN754410NE, U4 MCP9700A-E/TO

Commit message: plusieurs mises à jour
Parts:
- C4, C5, C6: footprint Capacitor_THT:C_Disc_D3.4mm_W2.1mm_P2.50mm -> Capacitor_SMD:C_0402_1005Metric
- D1, D2, D3, D4, D5: footprint BEAPER-Nano:LED_D3.0mm -> LED_SMD:LED_0603_1608Metric
- R1, R10, R11, R12, R13, R14, R15, R16, R17, R18, R19, R2, R20, R21, R22, R23, R24, R25, R26, R27, R28, R29, R3, R30, R4, R5, R6, R7, R8, R9: footprint Resistor_THT:R_Axial_DIN0207_L6.3mm_D2.5mm_P10.16mm_Horizontal -> Resistor_SMD:R_0603_1608Metric
Connections:
- net VBUS renamed /VBUS

Commit message: update avec les modules principaux
Parts:
- added GH1: MountingHole_2mm, MountingHole:MountingHole_2mm, F.Cu at (88.8, 36.0)
- added GH2: MountingHole_2mm, MountingHole:MountingHole_2mm, F.Cu at (105.5, 113.5)
- added GH3: MountingHole_2mm, MountingHole:MountingHole_2mm, F.Cu at (60.0, 113.5)
Other:
- board size 114.3 x 95.2 mm -> 65.5 x 100 mm
