File: BEAPER-Nano.kicad_sch (KiCad schematic)
At the start: 82 parts, among them CON1 Phoenix 1729160, J1 Digital, J2 Analog, J3 Conn_01x08, J4 QWIIC/JST SH, Q1 LTR-4206E, Q2 LTR-4206E, Q3 LTR-4206E, Q4 TEPT4400, SW1 RESET, SW2 SW_Push, SW3 SW_Push, SW4 SW_Push, SW5 SW_Push, U1 LM2940T-5.0, U2 74HCT541, U3 SN754410NE, U4 MCP9700A-E/TO

Commit message: Changement des pièces pour du smd
Parts:
- C4, C5, C6: footprint Capacitor_THT:C_Disc_D3.4mm_W2.1mm_P2.50mm -> Capacitor_SMD:C_0402_1005Metric
- D1, D2, D3, D4, D5: footprint BEAPER-Nano:LED_D3.0mm -> LED_SMD:LED_0603_1608Metric
- R1, R10, R11, R12, R13, R14, R15, R16, R17, R18, R19, R2, R20, R21, R22, R23, R24, R25, R26, R27, R28, R29, R3, R30, R4, R5, R6, R7, R8, R9: footprint Resistor_THT:R_Axial_DIN0207_L6.3mm_D2.5mm_P10.16mm_Horizontal -> Resistor_SMD:R_0603_1608Metric
Changed lines of the file:
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@@
 			)
 		)
-		(property "Footprint" "BEAPER-Nano:LED_D3.0mm"
+		(property "Footprint" "LED_SMD:LED_0603_1608Metric"
 			(at 41.91 251.46 0)
 			(hide yes)
@@
 			)
 		)
-		(property "Footprint" "BEAPER-Nano:LED_D3.0mm"
+		(property "Footprint" "LED_SMD:LED_0603_1608Metric"
 			(at 54.61 251.46 0)
 			(hide yes)
@@
 			)
 		)
-		(property "Footprint" "BEAPER-Nano:LED_D3.0mm"
+		(property "Footprint" "LED_SMD:LED_0603_1608Metric"
 			(at 67.31 251.46 0)
 			(hide yes)
@@
 			)
 		)
-		(property "Footprint" "BEAPER-Nano:LED_D3.0mm"
+		(property "Footprint" "LED_SMD:LED_0603_1608Metric"
 			(at 80.01 251.46 0)
 			(hide yes)
@@
 			)
 		)
-		(property "Footprint" "Resistor_THT:R_Axial_DIN0207_L6.3mm_D2.5mm_P10.16mm_Horizontal"
+		(property "Footprint" "Resistor_SMD:R_0603_1608Metric"
 			(at 121.92 32.258 90)
 			(hide yes)
@@
 			)
 		)
-		(property "Footprint" "Resistor_THT:R_Axial_DIN0207_L6.3mm_D2.5mm_P10.16mm_Horizontal"
+		(property "Footprint" "Resistor_SMD:R_0603_1608Metric"
 			(at 48.768 168.91 90)
 			(hide yes)
@@
 			)
 		)
-		(property "Footprint" "BEAPER-Nano:LED_D3.0mm"
+		(property "Footprint" "LED_SMD:LED_0603_1608Metric"
 			(at 46.99 177.8 0)
 			(hide yes)
@@
 			)
 		)
-		(property "Footprint" "Resistor_THT:R_Axial_DIN0207_L6.3mm_D2.5mm_P10.16mm_Horizontal"
+		(property "Footprint" "Resistor_SMD:R_0603_1608Metric"
 			(at 112.268 58.42 90)
 			(hide yes)
@@
 			)
 		)
-		(property "Footprint" "Resistor_THT:R_Axial_DIN0207_L6.3mm_D2.5mm_P10.16mm_Horizontal"
+		(property "Footprint" "Resistor_SMD:R_0603_1608Metric"
 			(at 347.472 39.37 90)
 			(hide yes)
@@
 			)
 		)
-		(property "Footprint" "Resistor_THT:R_Axial_DIN0207_L6.3mm_D2.5mm_P10.16mm_Horizontal"
+		(property "Footprint" "Resistor_SMD:R_0603_1608Metric"
 			(at 118.11 92.202 90)
 			(hide yes)
@@
 			)
 		)
-		(property "Footprint" "Resistor_THT:R_Axial_DIN0207_L6.3mm_D2.5mm_P10.16mm_Horizontal"
+		(property "Footprint" "Resistor_SMD:R_0603_1608Metric"
 			(at 118.11 104.902 90)
 			(hide yes)
@@
 			)
 		)
-		(property "Footprint" "Resistor_THT:R_Axial_DIN0207_L6.3mm_D2.5mm_P10.16mm_Horizontal"
+		(property "Footprint" "Resistor_SMD:R_0603_1608Metric"
 			(at 118.11 117.602 90)
 			(hide yes)
@@
 			)
 		)
-		(property "Footprint" "Resistor_THT:R_Axial_DIN0207_L6.3mm_D2.5mm_P10.16mm_Horizontal"
+		(property "Footprint" "Resistor_SMD:R_0603_1608Metric"
 			(at 118.11 130.302 90)
 			(hide yes)
@@
 			)
 		)
-		(property "Footprint" "Resistor_THT:R_Axial_DIN0207_L6.3mm_D2.5mm_P10.16mm_Horizontal"
+		(property "Footprint" "Resistor_SMD:R_0603_1608Metric"
 			(at 40.132 241.3 90)
 			(hide yes)
@@
 			)
 		)
-		(property "Footprint" "Resistor_THT:R_Axial_DIN0207_L6.3mm_D2.5mm_P10.16mm_Horizontal"
+		(property "Footprint" "Resistor_SMD:R_0603_1608Metric"
 			(at 52.832 241.3 90)
 			(hide yes)
@@
 			)
 		)
-		(property "Footprint" "Resistor_THT:R_Axial_DIN0207_L6.3mm_D2.5mm_P10.16mm_Horizontal"
+		(property "Footprint" "Resistor_SMD:R_0603_1608Metric"
 			(at 65.532 241.3 90)
 			(hide yes)
@@
 			)
 		)
-		(property "Footprint" "Resistor_THT:R_Axial_DIN0207_L6.3mm_D2.5mm_P10.16mm_Horizontal"
+		(property "Footprint" "Resistor_SMD:R_0603_1608Metric"
 			(at 78.232 241.3 90)
 			(hide yes)
@@
 			)
 		)
-		(property "Footprint" "Resistor_THT:R_Axial_DIN0207_L6.3mm_D2.5mm_P10.16mm_Horizontal"
+		(property "Footprint" "Resistor_SMD:R_0603_1608Metric"
 			(at 175.26 88.392 90)
 			(hide yes)
@@
 			)
 		)
-		(property "Footprint" "Resistor_THT:R_Axial_DIN0207_L6.3mm_D2.5mm_P10.16mm_Horizontal"
+		(property "Footprint" "Resistor_SMD:R_0603_1608Metric"
 			(at 175.26 99.822 90)
 			(hide yes)
@@
 			)
 		)
-		(property "Footprint" "Resistor_THT:R_Axial_DIN0207_L6.3mm_D2.5mm_P10.16mm_Horizontal"
+		(property "Footprint" "Resistor_SMD:R_0603_1608Metric"
 			(at 175.26 111.252 90)
 			(hide yes)
@@
 			)
 		)
-		(property "Footprint" "Resistor_THT:R_Axial_DIN0207_L6.3mm_D2.5mm_P10.16mm_Horizontal"
+		(property "Footprint" "Resistor_SMD:R_0603_1608Metric"
 			(at 175.26 122.682 90)
 			(hide yes)
@@
 			)
 		)
-		(property "Footprint" "Resistor_THT:R_Axial_DIN0207_L6.3mm_D2.5mm_P10.16mm_Horizontal"
+		(property "Footprint" "Resistor_SMD:R_0603_1608Metric"
 			(at 179.07 207.772 90)
 			(hide yes)
@@
 			)
 		)
-		(property "Footprint" "Capacitor_THT:C_Disc_D3.4mm_W2.1mm_P2.50mm"
+		(property "Footprint" "Capacitor_SMD:C_0402_1005Metric"
 			(at 244.8052 101.6 0)
 			(hide yes)
@@
 			)
 		)
-		(property "Footprint" "Resistor_THT:R_Axial_DIN0207_L6.3mm_D2.5mm_P10.16mm_Horizontal"
+		(property "Footprint" "Resistor_SMD:R_0603_1608Metric"
 			(at 178.562 45.72 90)
 			(hide yes)
@@
 			)
 		)
-		(property "Footprint" "Resistor_THT:R_Axial_DIN0207_L6.3mm_D2.5mm_P10.16mm_Horizontal"
+		(property "Footprint" "Resistor_SMD:R_0603_1608Metric"
 			(at 367.792 39.37 90)
 			(hide yes)
@@
 			)
 		)
-		(property "Footprint" "Resistor_THT:R_Axial_DIN0207_L6.3mm_D2.5mm_P10.16mm_Horizontal"
+		(property "Footprint" "Resistor_SMD:R_0603_1608Metric"
 			(at 393.192 100.33 90)
 			(hide yes)
@@
 			)
 		)
-		(property "Footprint" "Resistor_THT:R_Axial_DIN0207_L6.3mm_D2.5mm_P10.16mm_Horizontal"
+		(property "Footprint" "Resistor_SMD:R_0603_1608Metric"
 			(at 179.07 184.912 90)
 			(hide yes)
@@
 			)
 		)
-		(property "Footprint" "Resistor_THT:R_Axial_DIN0207_L6.3mm_D2.5mm_P10.16mm_Horizontal"
+		(property "Footprint" "Resistor_SMD:R_0603_1608Metric"
 			(at 235.712 200.66 90)
 			(hide yes)
@@
 			)
 		)
-		(property "Footprint" "Resistor_THT:R_Axial_DIN0207_L6.3mm_D2.5mm_P10.16mm_Horizontal"
+		(property "Footprint" "Resistor_SMD:R_0603_1608Metric"
 			(at 275.082 149.86 90)
 			(hide yes)
@@
 			)
 		)
-		(property "Footprint" "Resistor_THT:R_Axial_DIN0207_L6.3mm_D2.5mm_P10.16mm_Horizontal"
+		(property "Footprint" "Resistor_SMD:R_0603_1608Metric"
 			(at 391.922 39.37 90)
 			(hide yes)
@@
 			)
 		)
-		(property "Footprint" "Resistor_THT:R_Axial_DIN0207_L6.3mm_D2.5mm_P10.16mm_Horizontal"
+		(property "Footprint" "Resistor_SMD:R_0603_1608Metric"
 			(at 375.412 100.33 90)
 			(hide yes)
@@
 			)
 		)
-		(property "Footprint" "Resistor_THT:R_Axial_DIN0207_L6.3mm_D2.5mm_P10.16mm_Horizontal"
+		(property "Footprint" "Resistor_SMD:R_0603_1608Metric"
 			(at 236.982 43.18 90)
 			(hide yes)
@@
 			)
 		)
-		(property "Footprint" "Capacitor_THT:C_Disc_D3.4mm_W2.1mm_P2.50mm"
+		(property "Footprint" "Capacitor_SMD:C_0402_1005Metric"
 			(at 110.1852 204.47 0)
 			(hide yes)
@@
 			)
 		)
-		(property "Footprint" "Resistor_THT:R_Axial_DIN0207_L6.3mm_D2.5mm_P10.16mm_Horizontal"
+		(property "Footprint" "Resistor_SMD:R_0603_1608Metric"
 			(at 275.082 162.56 90)
 			(hide yes)
@@
 			)
 		)
-		(property "Footprint" "Resistor_THT:R_Axial_DIN0207_L6.3mm_D2.5mm_P10.16mm_Horizontal"
+		(property "Footprint" "Resistor_SMD:R_0603_1608Metric"
 			(at 179.07 196.342 90)
 			(hide yes)
@@
 			)
 		)
-		(property "Footprint" "Resistor_THT:R_Axial_DIN0207_L6.3mm_D2.5mm_P10.16mm_Horizontal"
+		(property "Footprint" "Resistor_SMD:R_0603_1608Metric"
 			(at 169.672 45.72 90)
 			(hide yes)
@@
 			)
 		)
-		(property "Footprint" "Resistor_THT:R_Axial_DIN0207_L6.3mm_D2.5mm_P10.16mm_Horizontal"
+		(property "Footprint" "Resistor_SMD:R_0603_1608Metric"
 			(at 179.07 173.482 90)
 			(hide yes)
@@
 			)
 		)
-		(property "Footprint" "Capacitor_THT:C_Disc_D3.4mm_W2.1mm_P2.50mm"
+		(property "Footprint" "Capacitor_SMD:C_0402_1005Metric"
 			(at 248.6152 204.47 0)
 			(hide yes)

Commit message: plusieurs mises à jour
Parts:
- removed D6, D7: OED-EL-1L2, BEAPER-Nano:LED_D5.0mm_Clear, symbol Device:LED
- removed H10, H9: Conn_01x03_Male, Connector_PinHeader_2.54mm:PinHeader_1x03_P2.54mm_Vertical, symbol Connector:Conn_01x03_Male
- removed H11, H12: Conn_01x04_Pin, Connector_PinHeader_2.54mm:PinHeader_1x04_P2.54mm_Vertical, symbol Connector:Conn_01x04_Pin
- removed J1: Digital, Connector_PinSocket_2.54mm:PinSocket_1x15_P2.54mm_Vertical, symbol Connector_Generic:Conn_01x15
- removed J2: Analog, Connector_PinSocket_2.54mm:PinSocket_1x15_P2.54mm_Vertical, symbol Connector_Generic:Conn_01x15
- removed JP1, JP2: ALS/LFS, Connector_PinHeader_2.54mm:PinHeader_1x03_P2.54mm_Vertical, symbol Jumper:Jumper_3_Open
- removed JP3, JP4: POT/VDIV, Connector_PinHeader_2.54mm:PinHeader_1x03_P2.54mm_Vertical, symbol Jumper:Jumper_3_Open
- removed Q1, Q2, Q3: LTR-4206E, BEAPER-Nano:LED_D3.0mm_IRBlack, symbol Sensor_Optical:TEPT4400
- removed Q4: TEPT4400, BEAPER-Nano:LED_D3.0mm_Clear, symbol Sensor_Optical:TEPT4400
- removed R18, R22, R23, R24: 4k7, Resistor_SMD:R_0603_1608Metric, symbol Device:R
- removed R20, R21: 100, Resistor_SMD:R_0603_1608Metric, symbol Device:R
- removed R25: 5.62k-1%, Resistor_SMD:R_0603_1608Metric, symbol Device:R
- removed R26: 1.37k-1%, Resistor_SMD:R_0603_1608Metric, symbol Device:R
- removed RV1, RV2: 10k, Potentiometer_THT:Potentiometer_Bourns_PTV09A-1_Single_Vertical, symbol Device:R_Potentiometer
- removed U3: SN754410NE, Package_DIP:DIP-16_W7.62mm, symbol Driver_Motor:SN754410NE
- added C10, C9: 100nF, Capacitor_SMD:C_0402_1005Metric, symbol Device:C
- added C11: 1uF, Capacitor_SMD:C_0402_1005Metric, symbol Device:C
- added C8: 470uF/16V, Capacitor_SMD:CP_Elec_8x10.5, symbol Device:C_Polarized
- added D8: SS54, Diode_SMD:D_SMA, symbol Device:D_Schottky
- added D9: SMAJ13A, Diode_SMD:D_SMA, symbol Device:D_TVS
- added F1: 3.5A, Fuse:Fuse_1206_3216Metric, symbol Device:Fuse
- added M1: Moteur 1 (MHDR1X6), Connector_PinHeader_2.54mm:PinHeader_1x06_P2.54mm_Vertical, symbol Connector_Generic:Conn_01x06
- added M2: Moteur 2 (MHDR1X6), Connector_PinHeader_2.54mm:PinHeader_1x06_P2.54mm_Vertical, symbol Connector_Generic:Conn_01x06
- added R31, R32, R33, R34: 51, Resistor_SMD:R_0603_1608Metric, symbol Device:R
- added R35: 100k, Resistor_SMD:R_0603_1608Metric, symbol Device:R
- added R36: 51k, Resistor_SMD:R_0603_1608Metric, symbol Device:R
- added U3: TB6612FNG, Package_SO:SSOP-24_5.3x8.2mm_P0.65mm, symbol Driver_Motor:TB6612FNG
- added U5: ESP32-S3-DevKitC-1-N16R8, BEAPER-Nano:ESP32-S3-DevKitC-1, symbol ESP32S3:ESP32-S3-DevKitC-1
- added U6: LSM6DS3TR-C, Package_LGA:LGA-14_3x2.5mm_P0.5mm_LayoutBorder3x4y, symbol Sensor_Motion:LSM6DS3
Connections:
- net +3V3: now also C10.1, C9.1, M1.3 (Pin_3), M2.3 (Pin_3), U5.L1 (3V3), U5.L2 (3V3), U6.12 (CS), U6.5 (VDDIO), U6.8 (VDD)
- net +5V: now also U3.15 (PWMB), U3.20 (VCC), U3.23 (PWMA), U5.L21 (5V)
- net A1: now also U4.2 (V_{OUT}), U5.R5 (GPIO2)
- net A6: now also U5.L6 (GPIO6)
- net A7: now also U5.L7 (GPIO7)
- net D10: now also U5.L16 (GPIO10)
- net D2: now also U5.L20 (GPIO14)
- net D3: now also U5.L8 (GPIO15)
- net D4: now also U5.L9 (GPIO16)
- net D5: now also U5.L10 (GPIO17)
- net D6: now also U5.L11 (GPIO18)
- net D7: now also U5.R18 (GPIO21)
- net D8: now also U5.R17 (GPIO47)
- net D9: now also U5.R10 (GPIO38)
- net GND: now also C10.2, C11.2, C8.2, C9.2, D9.1 (A1), M1.4 (Pin_4), M2.4 (Pin_4), R36.2, U3.10 (PGND2), U3.18 (GND), U3.3 (PGND1), U3.4 (PGND1), U3.9 (PGND2), U5.L22 (GND), U5.R1 (GND), U5.R21 (GND), U5.R22 (GND), U6.1 (SDO/SA0), U6.6 (GND), U6.7 (GND)
- net VCC: now also C8.1, D8.1 (K), R35.1, U3.13 (VM2), U3.14 (VM3), U3.24 (VM1); no longer CON1.1 (Pin_1)
- net ~{RST}: now also U5.L3 (RST)
- net MOTOR_STBY: now reaches R19.2
- net MOTOR_STBY: now also U3.19 (STBY)
- net M2_IN1: now reaches U2.12 (Y6)
- net M2_IN1: now also U3.17 (BIN1)
- net M2A: now reaches CON1.5 (Pin_5)
- net M2A: now also M2.6 (Pin_6), U3.11 (BO1), U3.12 (BO1)
- net M2B: now reaches CON1.6 (Pin_6)
- net M2B: now also M2.5 (Pin_5), U3.7 (BO2), U3.8 (BO2)
- net M2_IN2: now reaches U2.11 (Y7)
- net M2_IN2: now also U3.16 (BIN2)
- net M1_IN1: now reaches U2.14 (Y4)
- net M1_IN1: now also U3.21 (AIN1)
- net M1A: now reaches CON1.3 (Pin_3)
- net M1A: now also M1.6 (Pin_6), U3.1 (AO1), U3.2 (AO1)
- net M1B: now reaches CON1.4 (Pin_4)
- net M1B: now also M1.5 (Pin_5), U3.5 (AO2), U3.6 (AO2)
- net M1_IN2: now reaches U2.13 (Y5)
- net M1_IN2: now also U3.22 (AIN2)
- new net: CON1.1 (Pin_1), D9.2 (A2), F1.2
- new net: D8.2 (A), F1.1
- new net A4/SDA: U5.L12 (GPIO8), U6.14 (SDA)
- new net A5/SCL: U5.L15 (GPIO9), U6.13 (SCL)
- new net D0/RX0: U5.R3 (GPIO44/RX)
- new net D1/TX0: U5.R2 (GPIO43/TX)
- new net D11/COPI: U5.L17 (GPIO11)
- new net D12/CIPO: U5.L19 (GPIO13)
- new net D13/SCK: U5.L18 (GPIO12)
- new net ENC1A: R31.2, U5.R9 (GPIO39)
- new net ENC1A_H: M1.2 (Pin_2), R31.1
- new net ENC1B: R32.2, U5.R8 (GPIO40)
- new net ENC1B_H: M1.1 (Pin_1), R32.1
- new net ENC2A: R33.2, U5.R7 (GPIO41)
- new net ENC2A_H: M2.2 (Pin_2), R33.1
- new net ENC2B: R34.2, U5.R6 (GPIO42)
- new net ENC2B_H: M2.1 (Pin_1), R34.1
- new net VOL_BAT: C11.1, R35.2, R36.1, U5.L13 (GPIO3)
- no-connect marks 0 -> 18
Other:
- note removed: "Arduino Nano ESP32"

Commit message: update avec les modules principaux
Parts:
- removed R3, R4, R5, R6: 1k0, Resistor_SMD:R_0603_1608Metric, symbol Device:R
- removed SW2, SW3, SW4, SW5: SW_Push, Button_Switch_THT:SW_PUSH_6mm, symbol Switch:SW_Push
- added C12: 100nF, Capacitor_SMD:C_0402_1005Metric, symbol Device:C
- added J10: VL53L1X module, Connector_PinSocket_2.54mm:PinSocket_1x06_P2.54mm_Vertical, symbol Connector_Generic:Conn_01x06
- added J11: OLED I2C, Connector_PinSocket_2.54mm:PinSocket_1x04_P2.54mm_Vertical, symbol Connector_Generic:Conn_01x04
- added J12: PRGB (Auriga panel module), Connector_PinSocket_2.54mm:PinSocket_1x07_P2.54mm_Vertical, symbol Connector_Generic:Conn_01x07
- added J13: PG1 (GND support), Connector_PinSocket_2.54mm:PinSocket_1x02_P2.54mm_Vertical, symbol Connector_Generic:Conn_01x02
- added J14: PG2 (GND support), Connector_PinSocket_2.54mm:PinSocket_1x02_P2.54mm_Vertical, symbol Connector_Generic:Conn_01x02
- added J5: RJ25 port A, Connector_RJ:RJ12_Amphenol_54601-x06_Horizontal, symbol Connector:RJ25
- added J6: RJ25 port B, Connector_RJ:RJ12_Amphenol_54601-x06_Horizontal, symbol Connector:RJ25
- added J7: RJ25 port C, Connector_RJ:RJ12_Amphenol_54601-x06_Horizontal, symbol Connector:RJ25
- added J8, J9: QWIIC/JST SH, Connector_JST:JST_SH_SM04B-SRSS-TB_1x04-1MP_P1.00mm_Horizontal, symbol Connector_Generic:Conn_01x04
- added R37: 10k, Resistor_SMD:R_0603_1608Metric, symbol Device:R
- added R38: 15k, Resistor_SMD:R_0603_1608Metric, symbol Device:R
- added R39: 220, Resistor_SMD:R_0603_1608Metric, symbol Device:R
- added U7: 74AHCT1G125, Package_TO_SOT_SMD:SOT-23-5, symbol 74xGxx:74AHCT1G125
Connections:
- net +3V3: now also J10.1 (Pin_1), J11.2 (Pin_2), J8.2 (Pin_2), J9.2 (Pin_2)
- net +5V: now also C12.1, J12.7 (Pin_7), J5.4, J6.4, J7.4, U7.5 (VCC)
- net A4/SDA: now also J10.4 (Pin_4), J11.4 (Pin_4), J5.2, J6.2, J7.2, J8.3 (Pin_3), J9.3 (Pin_3)
- net A5/SCL: now also J10.3 (Pin_3), J11.3 (Pin_3), J5.1, J6.1, J7.1, J8.4 (Pin_4), J9.4 (Pin_4)
- net D10: now also J7.6
- net D9: now also J7.5
- net GND: now also C12.2, J10.2 (Pin_2), J11.1 (Pin_1), J12.6 (Pin_6), J13.1 (Pin_1), J13.2 (Pin_2), J14.1 (Pin_1), J14.2 (Pin_2), J5.3, J6.3, J7.3, J8.1 (Pin_1), J9.1 (Pin_1), R37.1, U7.1, U7.3 (GND)
- net VCC: now also J12.1 (Pin_1)
- net A2: now reaches U5.L4 (GPIO4)
- net A2: now also J12.3 (Pin_3)
- net A3: now reaches U5.L5 (GPIO5)
- net A3: now also J12.4 (Pin_4)
- net RGB_3V3: now reaches U5.R16 (GPIO48)
- net RGB_3V3: now also U7.2
- net PA_S1: now reaches U5.R4 (GPIO1)
- net PA_S1: now also J5.5
- net D0/RX0 renamed PB_S2
- net PB_S2: now also J6.6
- net D1/TX0 renamed PB_S1
- net PB_S1: now also J6.5
- net D2 renamed KEY_GPIO
- net KEY_GPIO: now also R37.2, R38.2
- net D3 renamed PA_S2
- net PA_S2: now also J5.6
- new net KEY: J12.2 (Pin_2), R38.1
- new net RGB: J12.5 (Pin_5), R39.2
- new net RGB_BUF: R39.1, U7.4
- no-connect marks 18 -> 16
