File: Beaper-Esp32s3.kicad_sch (KiCad schematic)
At the start: 80 parts, among them CON1 Phoenix 1729160, J10 VL53L1X module, J11 OLED I2C, J12 PRGB (Auriga panel module), J13 PG1 (GND support), J14 PG2 (GND support), J3 Conn_01x08, J4 QWIIC/JST SH, J5 RJ25 port A, J6 RJ25 port B, J7 RJ25 port C, J8 QWIIC/JST SH, J9 QWIIC/JST SH, M1 Moteur 1 (MHDR1X6), M2 Moteur 2 (MHDR1X6), SW1 RESET, U1 LM2940T-5.0, U2 74HCT541, U3 TB6612FNG, U4 MCP9700A-E/TO, U5 ESP32-S3-DevKitC-1-N16R8, U6 LSM6DS3TR-C, U7 74AHCT1G125

Commit message: Fusible de protection et datasheets
Parts:
- removed C1, C2: 10uF, Capacitor_THT:CP_Radial_D5.0mm_P2.50mm, symbol Device:C_Polarized
- removed U1: LM2940T-5.0, Package_TO_SOT_THT:TO-220-3_Horizontal_TabDown, symbol Regulator_Linear:LF50_TO220
- added C13: 10uF/50V, Capacitor_SMD:C_1206_3216Metric, symbol Device:C
- added C14, C15, C18: 100nF, Capacitor_SMD:C_0402_1005Metric, symbol Device:C
- added C16: 10nF, Capacitor_SMD:C_0402_1005Metric, symbol Device:C
- added C17: 470uF/16V, Capacitor_SMD:CP_Elec_8x10.5, symbol Device:C_Polarized
- added C19: 120pF, Capacitor_SMD:C_0402_1005Metric, symbol Device:C
- added C20: 68pF, Capacitor_SMD:C_0402_1005Metric, symbol Device:C
- added D10, D11, D13: SS34, Diode_SMD:D_SMA, symbol Device:D_Schottky
- added D12: SMAJ5.0CA, Diode_SMD:D_SMA, symbol Device:D_TVS
- added D14, D15, D16, D17: SMAJ12CA, Diode_SMD:D_SMA, symbol Device:D_TVS
- added F2: 3A, Fuse:Fuse_1206_3216Metric, symbol Device:Fuse
- added F3, F4, F5, F6: 1A PTC, Fuse:Fuse_1206_3216Metric, symbol Device:Fuse
- added FB1, FB2, FB3, FB4: 120R/2A, Inductor_SMD:L_0603_1608Metric, symbol Device:FerriteBead
- added L1: 6.8uH/4.5A, Inductor_SMD:L_Bourns_SRP7028A_7.3x6.6mm, symbol Device:L
- added R40: 10k, Resistor_SMD:R_0603_1608Metric, symbol Device:R
- added R41: 1.91k, Resistor_SMD:R_0603_1608Metric, symbol Device:R
- added R42: 30k, Resistor_SMD:R_0603_1608Metric, symbol Device:R
- added U1: TPS54331DDA, Package_SO:TI_SO-PowerPAD-8, symbol ESP32S3:TPS54331DDA
- C7: value 10uF -> 470uF/16V; footprint Capacitor_THT:CP_Radial_D5.0mm_P2.50mm -> Capacitor_SMD:CP_Elec_8x10.5; LCSC (none) -> C18221527
- C8: LCSC (none) -> C18221527
- D9: value SMAJ13A -> SMAJ13CA; LCSC (none) -> C19077534
Connections:
- net +5V: now also D11.1 (K), D12.2 (A2)
- net GND: now also C13.2, C14.2, C16.2, C17.2, C18.2, C19.2, C20.2, D10.2 (A), D12.1 (A1), D14.1 (A1), D15.1 (A1), D16.1 (A1), D17.1 (A1), R41.2, U1.7 (GND), U1.9 (PowerPAD)
- net M1A: now also F3.2; no longer U3.1 (AO1), U3.2 (AO1)
- net M1B: now also F4.2; no longer U3.5 (AO2), U3.6 (AO2)
- net M2A: now also F5.2; no longer U3.11 (BO1), U3.12 (BO1)
- net M2B: now also F6.2; no longer U3.7 (BO2), U3.8 (BO2)
- net VBAT: now reaches CON1.1 (Pin_1), D9.2 (A2), F1.2
- net VBAT: now also F2.1
- new net: F4.1, FB2.2
- new net: C20.1, R42.1, U1.6 (COMP)
- new net: D13.2 (A), F2.2
- new net: F3.1, FB1.2
- new net: C17.1, C18.1, D11.2 (A), L1.2, R40.1
- new net: C13.1, C14.1, D13.1 (K), U1.2 (VIN)
- new net: C15.1, U1.1 (BOOT)
- new net: C16.1, U1.4 (SS/TR)
- new net: C15.2, D10.1 (K), L1.1, U1.8 (PH)
- new net: F5.1, FB3.2
- new net: F6.1, FB4.2
- new net: C19.1, R42.2
- new net FB: R40.2, R41.1, U1.5 (VSENSE)
- new net M1A_D: D14.2 (A2), FB1.1, U3.1 (AO1), U3.2 (AO1)
- new net M1B_D: D15.2 (A2), FB2.1, U3.5 (AO2), U3.6 (AO2)
- new net M2A_D: D16.2 (A2), FB3.1, U3.11 (BO1), U3.12 (BO1)
- new net M2B_D: D17.2 (A2), FB4.1, U3.7 (BO2), U3.8 (BO2)
- no-connect marks 16 -> 17

Commit message: Ajout des jst-ph, ajustement des positions, headers i2c
Parts:
- removed CON1: Phoenix 1729160, TerminalBlock_Phoenix:TerminalBlock_Phoenix_MKDS-1,5-6-5.08_1x06_P5.08mm_Horizontal, symbol Connector:Screw_Terminal_01x06
- removed G1: mirobotech_logo, BEAPER-Nano:mirobo_logo_10, symbol UBMP4.1-rescue:mirobotech_logo-UBMP4
- removed H2: A6 (SONAR TRIG), Connector_PinHeader_2.54mm:PinHeader_1x03_P2.54mm_Vertical, symbol Connector:Conn_01x03_Male
- removed H3: A7 (SONAR ECHO), Connector_PinHeader_2.54mm:PinHeader_1x03_P2.54mm_Vertical, symbol Connector:Conn_01x03_Male
- removed H5: A4 (Servo 1), Connector_PinHeader_2.54mm:PinHeader_1x03_P2.54mm_Vertical, symbol Connector:Conn_01x03_Male
- removed H6: A5 (Servo 2), Connector_PinHeader_2.54mm:PinHeader_1x03_P2.54mm_Vertical, symbol Connector:Conn_01x03_Male
- removed R13, R14, R27, R28: 100, Resistor_SMD:R_0603_1608Metric, symbol Device:R
- added J1: DC jack 5.5x2.1, Connector_BarrelJack:BarrelJack_Horizontal, symbol Connector:Barrel_Jack
- added J15, J16: I2C (GND 3V3 SCL SDA), Connector_PinHeader_2.54mm:PinHeader_1x04_P2.54mm_Vertical, symbol Connector_Generic:Conn_01x04
- added JP1: I2C EXT 3V3/5V, Connector_PinHeader_2.54mm:PinHeader_1x03_P2.54mm_Vertical, symbol Connector_Generic:Conn_01x03
- added Q1, Q2, Q3, Q4, Q5, Q6, Q7, Q8: BSS138, Package_TO_SOT_SMD:SOT-23, symbol Transistor_FET:BSS138
- added R43, R44: 4.7k, Resistor_SMD:R_0603_1608Metric, symbol Device:R
- added R45, R46, R47, R48, R49, R50, R51, R52, R53, R54, R55, R56: 10k, Resistor_SMD:R_0603_1608Metric, symbol Device:R
- C17, C7, C8: footprint Capacitor_SMD:CP_Elec_8x10.5 -> Capacitor_SMD:CP_Elec_6.3x7.7; LCSC C18221527 -> C5354997
- C3: value 10uF -> 10uF/50V; footprint Capacitor_THT:CP_Radial_D5.0mm_P2.50mm -> Capacitor_SMD:C_1206_3216Metric; LCSC (none) -> C13585
- J9: value QWIIC/JST SH -> I2C (GND 3V3 SCL SDA); footprint Connector_JST:JST_SH_SM04B-SRSS-TB_1x04-1MP_P1.00mm_Horizontal -> Connector_PinHeader_2.54mm:PinHeader_1x04_P2.54mm_Vertical
- M1, M2: footprint Connector_PinHeader_2.54mm:PinHeader_1x06_P2.54mm_Vertical -> Connector_JST:JST_PH_S6B-PH-K_1x06_P2.00mm_Horizontal
- SW1: footprint Button_Switch_THT:SW_PUSH_6mm -> Button_Switch_SMD:SW_Push_1P1T-MP_NO_Horizontal_Alps_SKRTLAE010; LCSC (none) -> C110293
- U2: footprint Package_DIP:DIP-20_W7.62mm_Socket -> Package_SO:TSSOP-20_4.4x6.5mm_P0.65mm; LCSC (none) -> C53552921
- U4: value MCP9700A-E/TO -> MCP9700AT-E/TT; footprint Package_TO_SOT_THT:TO-92_HandSolder -> Package_TO_SOT_SMD:SOT-23; LCSC (none) -> C127949
Connections:
- net +3V3: now also J15.2 (Pin_2), J16.2 (Pin_2), JP1.1 (Pin_1), Q1.1 (G), Q2.1 (G), Q3.1 (G), Q4.1 (G), Q5.1 (G), Q6.1 (G), Q7.1 (G), Q8.1 (G), R45.2, R46.2, R47.2, R48.2, R49.2, R50.2
- net +5V: no longer J5.4, J6.4, J7.4
- net A4/SDA: now also Q1.2 (S); no longer J5.2, J6.2, J7.2, J8.3 (Pin_3), J9.3 (Pin_3)
- net A4/SDA: now also J8.3 (Pin_3), J9.4 (Pin_4), J15.4 (Pin_4), J16.4 (Pin_4)
- net A5/SCL: now also Q2.2 (S); no longer J5.1, J6.1, J7.1, J8.4 (Pin_4), J9.4 (Pin_4)
- net A5/SCL: now also J8.4 (Pin_4), J9.3 (Pin_3), J15.3 (Pin_3), J16.3 (Pin_3)
- net D10: now also Q8.2 (S), R50.1; no longer J7.6
- net D9: now also Q7.2 (S), R49.1; no longer J7.5
- net GND: now also J1.2, J15.1 (Pin_1), J16.1 (Pin_1)
- net PA_S1: now also Q3.2 (S), R45.1; no longer J5.5
- net PA_S2: now also Q4.2 (S), R46.1; no longer J5.6
- net PB_S1: now also Q5.2 (S), R47.1; no longer J6.5
- net PB_S2: now also Q6.2 (S), R48.1; no longer J6.6
- net VBAT: now also J1.1
- net 5V_P: now reaches C17.1, C18.1, D11.2 (A), L1.2, R40.1
- net 5V_P: now also J5.4, J6.4, J7.4, JP1.3 (Pin_3), R51.1, R52.1, R53.1, R54.1, R55.1, R56.1
- new net EXT_SCL: J5.1, J6.1, J7.1, Q2.3 (D), R44.2
- new net EXT_SDA: J5.2, J6.2, J7.2, Q1.3 (D), R43.2
- new net PA_S1_5V: J5.5, Q3.3 (D), R51.2
- new net PA_S2_5V: J5.6, Q4.3 (D), R52.2
- new net PB_S1_5V: J6.5, Q5.3 (D), R53.2
- new net PB_S2_5V: J6.6, Q6.3 (D), R54.2
- new net PC_S1_5V: J7.5, Q7.3 (D), R55.2
- new net PC_S2_5V: J7.6, Q8.3 (D), R56.2
- new net VI2C: JP1.2 (Pin_2), R43.1, R44.1
- no-connect marks 17 -> 19
Other:
- note added: "Makeblock RGB light sensor panel support"
- note removed: "Floor/line sensor LED"
- note removed: "Left floor sensor LED"
- note removed: "Left floor sensor phototransistor"
- note removed: "Left line sensor phototransistor"
- note removed: "Notes: 1. BEAPER Nano can be built in a simplified Educational Starter configuration using only the components not marked as optional. One or more optional analog input devices must be installed if using the analog input program in Introductory Programming Activity 5. 2. Headers H1-H4 can alternately be bridged with a 4-pin header socket to allow a 3.3V HC-SR04P SONAR distance sensing module to b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"
- note removed: "Optional ambient light sensor. (See note 4.)"
- note removed: "Optional analog potentiometer and external voltage divider. (See note 4.)"
- note removed: "Optional left floor sensor module. (See note 4.)"
- note removed: "Optional line sensor/ right floor sensor module. (See note 4.)"
- note removed: "Right floor/line sensor phototransistor"
- moved on the sheet: C10, C11, C12, C13, C14, C15, C16, C17, C18, C19, C20, C9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

Commit message: candidat pour pièces bien placées
Other:
- note added: "bidirectional logic level shifter"
- moved on the sheet: JP1, Q1, Q2, R43, R44

Commit message: Candidat avec J4 et J8 déplacé
Parts:
- U5: footprint BEAPER-Nano:ESP32-S3-DevKitC-1 -> BEAPER-Nano:ESP32-S3-DevKitC-1-2x22
Changed lines of the file:
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@@
 			)
 		)
-		(property "Footprint" "BEAPER-Nano:ESP32-S3-DevKitC-1"
+		(property "Footprint" "BEAPER-Nano:ESP32-S3-DevKitC-1-2x22"
 			(at 60.96 27.94 0)
 			(hide yes)
